File: src/stm32wb55vgy6-breakout.sch (EAGLE design)
At the start: 37 parts, among them J1 1x10, J10 PTH VERT MALE, J11 PTH VERT MALE, J2 1x10, J3 1x05 MALE VERT, J4 1x05 MALE VERT, J5 PTH VERT MALE, J6 PTH VERT MALE, J7 PTH VERT MALE, J8 PTH VERT MALE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

Commit message: [Rev 1] - Adjusted antenna microstrip width to more closely approximate a 50 ohm impedence.  Added LED power indicator to VCC.  Moved antenna circuitry to center of the board instead of the corner.
Parts:
- added LED1: BLUE, _leds:LED_SMD-0402_DISCRETE_BLUE
- added R1: 10K, _resistors:10KΩ_SMD-0402_1/16W-5%
Connections:
- new net N$1: LED1.K, R1.2
- net GND: now also R1.1
- net VCC: now also LED1.A
Changed lines of the file:
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@@
 <setting verticaltext="up"/>
 </settings>
-<grid distance="0.1" unitdist="inch" unit="inch" style="lines" multiple="1" display="yes" altdistance="0.01" altunitdist="inch" altunit="inch"/>
+<grid distance="0.1" unitdist="inch" unit="inch" style="lines" multiple="1" display="no" altdistance="0.01" altunitdist="inch" altunit="inch"/>
 <layers>
 <layer number="1" name="Top" color="4" fill="1" visible="no" active="no"/>
@@
 <part name="J3" library="_connectors" deviceset="1X05" device="_PTH_VERT_MALE_2.54MM" package3d_urn="urn:adsk.eagle:package:25810736/1" value="1x05 MALE VERT"/>
 <part name="J4" library="_connectors" deviceset="1X05" device="_PTH_VERT_MALE_2.54MM" package3d_urn="urn:adsk.eagle:package:25810736/1" value="1x05 MALE VERT"/>
+<part name="SUPPLY3" library="_power_symbols" deviceset="VCC" device=""/>
+<part name="LED1" library="_leds" deviceset="LED" device="_SMD-0402_DISCRETE_BLUE" package3d_urn="urn:adsk.eagle:package:2899303/3" value="BLUE"/>
+<part name="R1" library="_resistors" deviceset="10KΩ" device="_SMD-0402_1/16W-5%" package3d_urn="urn:adsk.eagle:package:2899165/1" value="10K"/>
+<part name="SUPPLY4" library="_power_symbols" deviceset="GND" device=""/>
 </parts>
 <sheets>
@@
 <attribute name="NAME" x="471.424" y="51.308" size="1.27" layer="95" font="vector" ratio="10" rot="MR0" align="bottom-right"/>
 </instance>
+<instance part="SUPPLY3" gate="VCC" x="513.08" y="88.9" smashed="yes"/>
+<instance part="LED1" gate="G$1" x="513.08" y="83.82" smashed="yes">
+<attribute name="NAME" x="513.334" y="84.074" size="1.27" layer="95" font="vector" ratio="10"/>
+<attribute name="VALUE" x="513.334" y="81.026" size="0.635" layer="96" font="vector" ratio="10" align="top-left"/>
+</instance>
+<instance part="R1" gate="G$1" x="513.08" y="71.12" smashed="yes" rot="R90">
+<attribute name="VALUE" x="514.223" y="71.12" size="0.635" layer="96" font="vector" ratio="10" rot="R90" align="top-center"/>
+<attribute name="NAME" x="511.9624" y="71.12" size="1.27" layer="95" font="vector" ratio="10" rot="R90" align="bottom-center"/>
+</instance>
+<instance part="SUPPLY4" gate="GND" x="513.08" y="60.96" smashed="yes"/>
 </instances>
 <busses>
@@
 <pinref part="SW1" gate="G$1" pin="1"/>
 <wire x1="25.4" y1="203.2" x2="25.4" y2="208.28" width="0.1524" layer="91"/>
+</segment>
+<segment>
+<pinref part="R1" gate="G$1" pin="1"/>
+<pinref part="SUPPLY4" gate="GND" pin="GND"/>
+<wire x1="513.08" y1="63.5" x2="513.08" y2="66.04" width="0.1524" layer="91"/>
 </segment>
 </net>
@@
 <wire x1="464.82" y1="63.5" x2="464.82" y2="91.44" width="0.1524" layer="91"/>
 </segment>
+<segment>
+<pinref part="LED1" gate="G$1" pin="A"/>
+<pinref part="SUPPLY3" gate="VCC" pin="VCC"/>
+<wire x1="513.08" y1="86.36" x2="513.08" y2="88.9" width="0.1524" layer="91"/>
+</segment>
 </net>
 <net name="N$12" class="0">
@@
 </segment>
 </net>
+<net name="N$1" class="0">
+<segment>
+<pinref part="LED1" gate="G$1" pin="K"/>
+<pinref part="R1" gate="G$1" pin="2"/>
+<wire x1="513.08" y1="76.2" x2="513.08" y2="78.74" width="0.1524" layer="91"/>
+</segment>
+</net>
